File: Detector de Metais/4011.sch (KiCad schematic (older format))
At the start: 8 parts, among them U5 4011

Commit message: Atualizando simbolos e criando footprint
Parts:
- C11, C12, C13: footprint (none) -> Capacitor_THT:C_Disc_D9.0mm_W5.0mm_P5.00mm
- R11, R13: footprint (none) -> Resistor_THT:R_Axial_DIN0204_L3.6mm_D1.6mm_P1.90mm_Vertical
- U5: footprint (none) -> Package_DIP:DIP-14_W7.62mm_Socket_LongPads
Changed lines of the file:
@@
 F 0 "U5" H 3100 3600 50  0000 C CNN
 F 1 "4011" H 3100 3500 50  0000 C CNN
-F 2 "" H 3100 3550 60  0001 C CNN
+F 2 "Package_DIP:DIP-14_W7.62mm_Socket_LongPads" H 3100 3550 60  0001 C CNN
 F 3 "" H 3100 3550 60  0001 C CNN
 	1    3100 3550
@@
 F 0 "U5" H 4950 3600 50  0000 C CNN
 F 1 "4011" H 4950 3500 50  0000 C CNN
-F 2 "" H 4950 3550 60  0001 C CNN
+F 2 "Package_DIP:DIP-14_W7.62mm_Socket_LongPads" H 4950 3550 60  0001 C CNN
 F 3 "" H 4950 3550 60  0001 C CNN
 	2    4950 3550
@@
 F 0 "U5" H 6650 3600 50  0000 C CNN
 F 1 "4011" H 6650 3500 50  0000 C CNN
-F 2 "" H 6650 3550 60  0001 C CNN
+F 2 "Package_DIP:DIP-14_W7.62mm_Socket_LongPads" H 6650 3550 60  0001 C CNN
 F 3 "" H 6650 3550 60  0001 C CNN
 	3    6650 3550
@@
 F 0 "U5" H 8550 3600 50  0000 C CNN
 F 1 "4011" H 8550 3500 50  0000 C CNN
-F 2 "" H 8550 3550 60  0001 C CNN
+F 2 "Package_DIP:DIP-14_W7.62mm_Socket_LongPads" H 8550 3550 60  0001 C CNN
 F 3 "" H 8550 3550 60  0001 C CNN
 	4    8550 3550
@@
 F 0 "R11" V 3630 2950 50  0000 C CNN
 F 1 "33k" V 3550 2950 50  0000 C CNN
-F 2 "" V 3480 2950 50  0001 C CNN
+F 2 "Resistor_THT:R_Axial_DIN0204_L3.6mm_D1.6mm_P1.90mm_Vertical" V 3480 2950 50  0001 C CNN
 F 3 "" H 3550 2950 50  0001 C CNN
 	1    3550 2950
@@
 F 0 "C12" H 4075 3650 50  0000 L CNN
 F 1 "1nF" H 4075 3450 50  0000 L CNN
-F 2 "" H 4088 3400 50  0001 C CNN
+F 2 "Capacitor_THT:C_Disc_D9.0mm_W5.0mm_P5.00mm" H 4088 3400 50  0001 C CNN
 F 3 "" H 4050 3550 50  0001 C CNN
 	1    4050 3550
@@
 F 0 "C11" H 4675 3250 50  0000 L CNN
 F 1 "1nF" H 4675 3050 50  0000 L CNN
-F 2 "" H 4688 3000 50  0001 C CNN
+F 2 "Capacitor_THT:C_Disc_D9.0mm_W5.0mm_P5.00mm" H 4688 3000 50  0001 C CNN
 F 3 "" H 4650 3150 50  0001 C CNN
 	1    4650 3150
@@
 F 0 "R13" V 4380 4050 50  0000 C CNN
 F 1 "33k" V 4300 4050 50  0000 C CNN
-F 2 "" V 4230 4050 50  0001 C CNN
+F 2 "Resistor_THT:R_Axial_DIN0204_L3.6mm_D1.6mm_P1.90mm_Vertical" V 4230 4050 50  0001 C CNN
 F 3 "" H 4300 4050 50  0001 C CNN
 	1    4300 4050
@@
 F 0 "C13" H 7675 3650 50  0000 L CNN
 F 1 "1nF" H 7675 3450 50  0000 L CNN
-F 2 "" H 7688 3400 50  0001 C CNN
+F 2 "Capacitor_THT:C_Disc_D9.0mm_W5.0mm_P5.00mm" H 7688 3400 50  0001 C CNN
 F 3 "" H 7650 3550 50  0001 C CNN
 	1    7650 3550
