File: Detector de Metais/555+357.sch (KiCad schematic (older format))
At the start: 25 parts, among them Q3 BC807-40 ou BC327, Q4 BD911, U6 NE555, U7 TL071

Commit message: Atualizando simbolos e criando footprint
Parts:
- C14: footprint (none) -> Capacitor_THT:C_Disc_D9.0mm_W5.0mm_P5.00mm
- C15, C17, C18, C19, C20: footprint (none) -> Capacitor_THT:C_Disc_D6.0mm_W2.5mm_P5.00mm
- C16, C21: footprint (none) -> Capacitor_THT:C_Disc_D4.3mm_W1.9mm_P5.00mm
- DZ1: footprint (none) -> Diode_THT:D_A-405_P2.54mm_Vertical_AnodeUp
- L1: footprint (none) -> Connector_BarrelJack:BarrelJack_Horizontal
- PTR2: footprint (none) -> Potentiometer_THT:Potentiometer_ACP_CA9-H3,8_Horizontal
- Q3: footprint TO_SOT_Packages_SMD:SOT-23 -> Package_TO_SOT_THT:TO-92L
- Q4: footprint TO_SOT_Packages_THT:TO-220_Vertical -> Package_TO_SOT_THT:TO-220-3_Vertical
- R18, R24: footprint (none) -> Resistor_THT:R_Axial_DIN0204_L3.6mm_D1.6mm_P1.90mm_Vertical
- R20: footprint (none) -> Resistor_THT:R_Axial_DIN0207_L6.3mm_D2.5mm_P5.08mm_Vertical
- R22: P/N MC01W08051820K -> MC01W0805110K
- U6: footprint (none) -> Package_SO:HTSOP-8-1EP_3.9x4.9mm_P1.27mm_EP2.4x3.2mm
- U7: footprint (none) -> Package_DIP:DIP-8_W7.62mm_LongPads
Changed lines of the file:
@@
 F 0 "U6" H 2200 3650 50  0000 L CNN
 F 1 "NE555" H 2200 2950 50  0000 L CNN
-F 2 "" H 2600 3300 50  0001 C CNN
+F 2 "Package_SO:HTSOP-8-1EP_3.9x4.9mm_P1.27mm_EP2.4x3.2mm" H 2600 3300 50  0001 C CNN
 F 3 "" H 2600 3300 50  0001 C CNN
 	1    2600 3300
@@
 F 0 "L1" V 5900 4200 50  0000 C CNN
 F 1 "Bobina" V 6025 4200 50  0000 C CNN
-F 2 "" H 5950 4200 50  0001 C CNN
-F 3 "" H 5950 4200 50  0001 C CNN
+F 2 "Connector_BarrelJack:BarrelJack_Horizontal" H 5950 4200 50  0001 C CNN
+F 3 "Fazer" H 5950 4200 50  0001 C CNN
 	1    5950 4200
 	1    0    0    -1
@@
 F 0 "DZ1" H 7050 4000 50  0000 C CNN
 F 1 "3,3v" H 7050 3800 50  0000 C CNN
-F 2 "" H 7050 3900 50  0001 C CNN
+F 2 "Diode_THT:D_A-405_P2.54mm_Vertical_AnodeUp" H 7050 3900 50  0001 C CNN
 F 3 "" H 7050 3900 50  0001 C CNN
 	1    7050 3900
@@
 F 0 "Q4" H 6400 4875 50  0000 L CNN
 F 1 "BD911" H 6400 4800 50  0000 L CNN
-F 2 "TO_SOT_Packages_THT:TO-220_Vertical" H 6400 4725 50  0001 L CIN
-F 3 "" H 6150 4800 50  0001 L CNN
+F 2 "Package_TO_SOT_THT:TO-220-3_Vertical" H 6400 4725 50  0001 L CIN
+F 3 "Falta" H 6150 4800 50  0001 L CNN
 	1    6150 4800
 	1    0    0    -1
@@
 F 0 "Q3" H 4800 4250 50  0000 L CNN
 F 1 "BC807-40 ou BC327" V 5100 3600 50  0000 L CNN
-F 2 "TO_SOT_Packages_SMD:SOT-23" H 5100 4025 50  0001 L CIN
+F 2 "Package_TO_SOT_THT:TO-92L" H 5100 4025 50  0001 L CIN
 F 3 "" H 4900 4100 50  0001 L CNN
 	1    4900 4100
@@
 F 0 "C16" H 1925 4050 50  0000 L CNN
 F 1 "100nF" H 1925 3850 50  0000 L CNN
-F 2 "" H 1938 3800 50  0001 C CNN
+F 2 "Capacitor_THT:C_Disc_D4.3mm_W1.9mm_P5.00mm" H 1938 3800 50  0001 C CNN
 F 3 "" H 1900 3950 50  0001 C CNN
 	1    1900 3950
@@
 F 0 "C15" H 1625 4050 50  0000 L CNN
 F 1 "200nF" H 1625 3850 50  0000 L CNN
-F 2 "" H 1638 3800 50  0001 C CNN
-F 3 "" H 1600 3950 50  0001 C CNN
+F 2 "Capacitor_THT:C_Disc_D6.0mm_W2.5mm_P5.00mm" H 1638 3800 50  0001 C CNN
+F 3 "Falta" H 1600 3950 50  0001 C CNN
 	1    1600 3950
 	1    0    0    -1
@@
 F 0 "PTR2" V 3175 2550 50  0000 C CNN
 F 1 "100k" V 3250 2550 50  0000 C CNN
-F 2 "" H 3350 2550 50  0001 C CNN
+F 2 "Potentiometer_THT:Potentiometer_ACP_CA9-H3,8_Horizontal" H 3350 2550 50  0001 C CNN
 F 3 "" H 3350 2550 50  0001 C CNN
 	1    3350 2550
@@
 F 0 "R18" V 4280 4100 50  0000 C CNN
 F 1 "1,2k" V 4200 4100 50  0000 C CNN
-F 2 "" V 4130 4100 50  0001 C CNN
+F 2 "Resistor_THT:R_Axial_DIN0204_L3.6mm_D1.6mm_P1.90mm_Vertical" V 4130 4100 50  0001 C CNN
 F 3 "" H 4200 4100 50  0001 C CNN
 	1    4200 4100
@@
 F 0 "C14" H 5575 3250 50  0000 L CNN
 F 1 "1nF" H 5575 3050 50  0000 L CNN
-F 2 "" H 5588 3000 50  0001 C CNN
+F 2 "Capacitor_THT:C_Disc_D9.0mm_W5.0mm_P5.00mm" H 5588 3000 50  0001 C CNN
 F 3 "" H 5550 3150 50  0001 C CNN
 	1    5550 3150
@@
 F 0 "R24" V 5730 5050 50  0000 C CNN
 F 1 "150" V 5650 5050 50  0000 C CNN
-F 2 "" V 5580 5050 50  0001 C CNN
+F 2 "Resistor_THT:R_Axial_DIN0204_L3.6mm_D1.6mm_P1.90mm_Vertical" V 5580 5050 50  0001 C CNN
 F 3 "" H 5650 5050 50  0001 C CNN
 	1    5650 5050
@@
 F 0 "R20" V 6930 4450 50  0000 C CNN
 F 1 "200/0,5W" V 6750 4450 50  0000 C CNN
-F 2 "" V 6780 4450 50  0001 C CNN
+F 2 "Resistor_THT:R_Axial_DIN0207_L6.3mm_D2.5mm_P5.08mm_Vertical" V 6780 4450 50  0001 C CNN
 F 3 "" H 6850 4450 50  0001 C CNN
 	1    6850 4450
@@
 F 0 "C18" H 6625 4100 50  0000 L CNN
 F 1 "47nF" H 6625 3900 50  0000 L CNN
-F 2 "" H 6638 3850 50  0001 C CNN
-F 3 "" H 6600 4000 50  0001 C CNN
+F 2 "Capacitor_THT:C_Disc_D6.0mm_W2.5mm_P5.00mm" H 6638 3850 50  0001 C CNN
+F 3 "Falta" H 6600 4000 50  0001 C CNN
 	1    6600 4000
 	1    0    0    -1
@@
 F 0 "C20" V 7450 4450 50  0000 L CNN
 F 1 "10uF/16V" V 7150 4250 50  0000 L CNN
-F 2 "" H 7338 4300 50  0001 C CNN
-F 3 "" H 7300 4450 50  0001 C CNN
+F 2 "Capacitor_THT:C_Disc_D6.0mm_W2.5mm_P5.00mm" H 7338 4300 50  0001 C CNN
+F 3 "Falta" H 7300 4450 50  0001 C CNN
 	1    7300 4450
 	0    -1   -1   0
@@
 F 2 "Resistor_SMD:R_0805_2012Metric_Pad1.15x1.40mm_HandSolder" V 8230 4950 50  0001 C CNN
 F 3 "" H 8300 4950 50  0001 C CNN
-F 4 "MC01W08051820K" H 8300 4950 50  0001 C CNN "P/N"
+F 4 "MC01W0805110K" H 8300 4950 50  0001 C CNN "P/N"
 	1    8300 4950
 	0    1    1    0
@@
 F 0 "U7" H 8200 4600 50  0000 L CNN
 F 1 "TL071" H 8200 4500 50  0000 L CNN
-F 2 "" H 8250 4400 50  0001 C CNN
+F 2 "Package_DIP:DIP-8_W7.62mm_LongPads" H 8250 4400 50  0001 C CNN
 F 3 "" H 8350 4500 50  0001 C CNN
 	1    8200 4350
@@
 F 0 "C17" H 8475 4050 50  0000 L CNN
 F 1 "10pF" V 8300 3850 50  0000 L CNN
-F 2 "" H 8488 3800 50  0001 C CNN
-F 3 "" H 8450 3950 50  0001 C CNN
+F 2 "Capacitor_THT:C_Disc_D6.0mm_W2.5mm_P5.00mm" H 8488 3800 50  0001 C CNN
+F 3 "Falta" H 8450 3950 50  0001 C CNN
 	1    8450 3950
 	0    1    1    0
@@
 F 0 "C19" H 8925 4450 50  0000 L CNN
 F 1 "3,3pF" V 8750 4250 50  0000 L CNN
-F 2 "" H 8938 4200 50  0001 C CNN
-F 3 "" H 8900 4350 50  0001 C CNN
+F 2 "Capacitor_THT:C_Disc_D6.0mm_W2.5mm_P5.00mm" H 8938 4200 50  0001 C CNN
+F 3 "Falta" H 8900 4350 50  0001 C CNN
 	1    8900 4350
 	0    1    1    0
@@
 F 0 "C21" H 9625 4700 50  0000 L CNN
 F 1 "100nF" V 9450 4500 50  0000 L CNN
-F 2 "" H 9638 4450 50  0001 C CNN
+F 2 "Capacitor_THT:C_Disc_D4.3mm_W1.9mm_P5.00mm" H 9638 4450 50  0001 C CNN
 F 3 "" H 9600 4600 50  0001 C CNN
 	1    9600 4600
