File: Detector de Metais/555+Audio.sch (KiCad schematic (older format))
At the start: 13 parts, among them Q5 BD140, U8 NE555

Commit message: Atualizando simbolos e criando footprint
Parts:
- C22, C23: footprint (none) -> Capacitor_THT:CP_Axial_L10.0mm_D6.0mm_P15.00mm_Horizontal
- C24, C26: footprint (none) -> Capacitor_THT:C_Disc_D4.3mm_W1.9mm_P5.00mm
- C25: footprint (none) -> Capacitor_THT:C_Disc_D6.0mm_W4.4mm_P5.00mm
- C27: footprint (none) -> Capacitor_THT:CP_Radial_D6.3mm_P2.50mm
- POT3: footprint (none) -> Potentiometer_THT:Potentiometer_Vishay_148-149_Single_Horizontal
- Q5: footprint TO_SOT_Packages_THT:TO-126_Vertical -> Package_TO_SOT_THT:TO-126-3_Vertical
- R26: footprint (none) -> Resistor_THT:R_Axial_DIN0204_L3.6mm_D1.6mm_P1.90mm_Vertical
- SP1: footprint (none) -> Connector_PinHeader_1.27mm:PinHeader_1x02_P1.27mm_Horizontal
- U8: footprint (none) -> Package_SO:HTSOP-8-1EP_3.9x4.9mm_P1.27mm_EP2.4x3.2mm
Changed lines of the file:
@@
 F 0 "Q5" H 7450 4275 50  0000 L CNN
 F 1 "BD140" H 7450 4200 50  0000 L CNN
-F 2 "TO_SOT_Packages_THT:TO-126_Vertical" H 7450 4125 50  0001 L CIN
+F 2 "Package_TO_SOT_THT:TO-126-3_Vertical" H 7450 4125 50  0001 L CIN
 F 3 "" H 7250 4200 50  0001 L CNN
 	1    7250 4200
@@
 F 0 "R26" V 5480 3950 50  0000 C CNN
 F 1 "2,4k" V 5400 3950 50  0000 C CNN
-F 2 "" V 5330 3950 50  0001 C CNN
-F 3 "" H 5400 3950 50  0001 C CNN
+F 2 "Resistor_THT:R_Axial_DIN0204_L3.6mm_D1.6mm_P1.90mm_Vertical" V 5330 3950 50  0001 C CNN
+F 3 "Falta" H 5400 3950 50  0001 C CNN
 	1    5400 3950
 	0    1    1    0
@@
 F 0 "C25" H 3475 3850 50  0000 L CNN
 F 1 "220nF" H 3200 3650 50  0000 L CNN
-F 2 "" H 3488 3600 50  0001 C CNN
+F 2 "Capacitor_THT:C_Disc_D6.0mm_W4.4mm_P5.00mm" H 3488 3600 50  0001 C CNN
 F 3 "" H 3450 3750 50  0001 C CNN
 	1    3450 3750
@@
 F 0 "C26" H 3825 3850 50  0000 L CNN
 F 1 "100nF" V 3950 3650 50  0000 L CNN
-F 2 "" H 3838 3600 50  0001 C CNN
+F 2 "Capacitor_THT:C_Disc_D4.3mm_W1.9mm_P5.00mm" H 3838 3600 50  0001 C CNN
 F 3 "" H 3800 3750 50  0001 C CNN
 	1    3800 3750
@@
 F 0 "C27" H 3375 4350 50  0000 L CNN
 F 1 "100uF/25V" V 3200 4150 50  0000 L CNN
-F 2 "" H 3388 4100 50  0001 C CNN
+F 2 "Capacitor_THT:CP_Radial_D6.3mm_P2.50mm" H 3388 4100 50  0001 C CNN
 F 3 "" H 3350 4250 50  0001 C CNN
 	1    3350 4250
@@
 F 0 "POT3" V 6275 3100 50  0000 C CNN
 F 1 "10k" V 6350 3100 50  0000 C CNN
-F 2 "" H 6450 3100 50  0001 C CNN
+F 2 "Potentiometer_THT:Potentiometer_Vishay_148-149_Single_Horizontal" H 6450 3100 50  0001 C CNN
 F 3 "" H 6450 3100 50  0001 C CNN
 	1    6450 3100
@@
 F 0 "SP1" H 7650 2850 50  0000 R CNN
 F 1 "Speaker 8ohm 0,5W" H 8150 3250 50  0000 R CNN
-F 2 "" H 7700 2850 50  0001 C CNN
+F 2 "Connector_PinHeader_1.27mm:PinHeader_1x02_P1.27mm_Horizontal" H 7700 2850 50  0001 C CNN
 F 3 "" H 7690 3000 50  0001 C CNN
 	1    7700 3050
@@
 F 0 "C22" H 8325 3700 50  0000 L CNN
 F 1 "1000uF/16V" V 8150 3400 50  0000 L CNN
-F 2 "" H 8338 3450 50  0001 C CNN
+F 2 "Capacitor_THT:CP_Axial_L10.0mm_D6.0mm_P15.00mm_Horizontal" H 8338 3450 50  0001 C CNN
 F 3 "" H 8300 3600 50  0001 C CNN
 	1    8300 3600
@@
 F 0 "C23" H 8675 3700 50  0000 L CNN
 F 1 "1000uF/16V" V 8500 3400 50  0000 L CNN
-F 2 "" H 8688 3450 50  0001 C CNN
+F 2 "Capacitor_THT:CP_Axial_L10.0mm_D6.0mm_P15.00mm_Horizontal" H 8688 3450 50  0001 C CNN
 F 3 "" H 8650 3600 50  0001 C CNN
 	1    8650 3600
@@
 F 0 "C24" H 8975 3700 50  0000 L CNN
 F 1 "100nF" V 8900 3650 50  0000 L CNN
-F 2 "" H 8988 3450 50  0001 C CNN
+F 2 "Capacitor_THT:C_Disc_D4.3mm_W1.9mm_P5.00mm" H 8988 3450 50  0001 C CNN
 F 3 "" H 8950 3600 50  0001 C CNN
 	1    8950 3600
@@
 F 0 "U8" H 4200 4100 50  0000 L CNN
 F 1 "NE555" H 4200 3400 50  0000 L CNN
-F 2 "" H 4600 3750 50  0001 C CNN
+F 2 "Package_SO:HTSOP-8-1EP_3.9x4.9mm_P1.27mm_EP2.4x3.2mm" H 4600 3750 50  0001 C CNN
 F 3 "" H 4600 3750 50  0001 C CNN
 	1    4600 3750
