File: Detector de Metais/Fonte.sch (KiCad schematic (older format))
At the start: 19 parts, among them J1 BARREL_JACK, U1 7805, U2 NE555, U3 7905

Commit message: Atualizando simbolos e criando footprint
Parts:
- C1, C7, C8: footprint (none) -> Capacitor_THT:CP_Radial_D5.0mm_P2.50mm
- C2, C4: footprint (none) -> Capacitor_THT:C_Disc_D4.3mm_W1.9mm_P5.00mm
- C5, C6: footprint (none) -> Capacitor_THT:CP_Radial_D6.3mm_P2.50mm
- C9: footprint (none) -> Capacitor_THT:C_Disc_D6.0mm_W2.5mm_P5.00mm
- D1, D2, D3, D4: footprint (none) -> Diode_THT:D_DO-41_SOD81_P2.54mm_Vertical_AnodeUp
- U1, U3: footprint (none) -> Package_TO_SOT_THT:TO-220-3_Vertical
- U2: footprint (none) -> Package_SO:HTSOP-8-1EP_3.9x4.9mm_P1.27mm_EP2.4x3.2mm
Changed lines of the file:
@@
 F 0 "U2" H 4150 3600 50  0000 L CNN
 F 1 "NE555" H 4150 2900 50  0000 L CNN
-F 2 "" H 4550 3250 50  0001 C CNN
+F 2 "Package_SO:HTSOP-8-1EP_3.9x4.9mm_P1.27mm_EP2.4x3.2mm" H 4550 3250 50  0001 C CNN
 F 3 "" H 4550 3250 50  0001 C CNN
 	1    4550 3250
@@
 F 0 "C9" H 2775 6000 50  0000 L CNN
 F 1 "22uF" H 2775 5800 50  0000 L CNN
-F 2 "" H 2788 5750 50  0001 C CNN
-F 3 "" H 2750 5900 50  0001 C CNN
+F 2 "Capacitor_THT:C_Disc_D6.0mm_W2.5mm_P5.00mm" H 2788 5750 50  0001 C CNN
+F 3 "Falta" H 2750 5900 50  0001 C CNN
 	1    2750 5900
 	1    0    0    -1
@@
 F 0 "D1" H 7050 4250 50  0000 C CNN
 F 1 "1N4004" H 7050 4050 50  0000 C CNN
-F 2 "" H 7050 4150 50  0001 C CNN
+F 2 "Diode_THT:D_DO-41_SOD81_P2.54mm_Vertical_AnodeUp" H 7050 4150 50  0001 C CNN
 F 3 "" H 7050 4150 50  0001 C CNN
 F 4 "MC01W08051180R" H 7050 4150 50  0001 C CNN "P/N"
@@
 F 0 "U3" H 2300 5955 50  0000 C CNN
 F 1 "7905" H 2150 6350 50  0000 C CNN
-F 2 "" H 2150 6150 50  0001 C CNN
+F 2 "Package_TO_SOT_THT:TO-220-3_Vertical" H 2150 6150 50  0001 C CNN
 F 3 "" H 2150 6150 50  0001 C CNN
 	1    2150 6150
@@
 F 0 "U1" H 9150 3004 50  0000 C CNN
 F 1 "7805" H 9000 3400 50  0000 C CNN
-F 2 "" H 9000 3200 50  0001 C CNN
+F 2 "Package_TO_SOT_THT:TO-220-3_Vertical" H 9000 3200 50  0001 C CNN
 F 3 "" H 9000 3200 50  0001 C CNN
 	1    9000 3200
@@
 F 0 "C4" H 3925 4000 50  0000 L CNN
 F 1 "100nF" H 3925 3800 50  0000 L CNN
-F 2 "" H 3938 3750 50  0001 C CNN
+F 2 "Capacitor_THT:C_Disc_D4.3mm_W1.9mm_P5.00mm" H 3938 3750 50  0001 C CNN
 F 3 "" H 3900 3900 50  0001 C CNN
 	1    3900 3900
@@
 F 1 "10nF" H 3625 3800 50  0000 L CNN
 F 2 "" H 3638 3750 50  0001 C CNN
-F 3 "" H 3600 3900 50  0001 C CNN
+F 3 "Falta" H 3600 3900 50  0001 C CNN
 	1    3600 3900
 	1    0    0    -1
@@
 F 0 "C7" H 6325 4550 50  0000 L CNN
 F 1 "22uF/16V" V 6150 4300 50  0000 L CNN
-F 2 "" H 6338 4300 50  0001 C CNN
+F 2 "Capacitor_THT:CP_Radial_D5.0mm_P2.50mm" H 6338 4300 50  0001 C CNN
 F 3 "" H 6300 4450 50  0001 C CNN
 	1    6300 4450
@@
 F 0 "C8" H 6325 4950 50  0000 L CNN
 F 1 "22uF/16V" V 6450 4650 50  0000 L CNN
-F 2 "" H 6338 4700 50  0001 C CNN
+F 2 "Capacitor_THT:CP_Radial_D5.0mm_P2.50mm" H 6338 4700 50  0001 C CNN
 F 3 "" H 6300 4850 50  0001 C CNN
 	1    6300 4850
@@
 F 0 "D3" H 7050 4950 50  0000 C CNN
 F 1 "1N4004" H 7050 4750 50  0000 C CNN
-F 2 "" H 7050 4850 50  0001 C CNN
+F 2 "Diode_THT:D_DO-41_SOD81_P2.54mm_Vertical_AnodeUp" H 7050 4850 50  0001 C CNN
 F 3 "" H 7050 4850 50  0001 C CNN
 F 4 "MC01W08051180R" H 7050 4850 50  0001 C CNN "P/N"
@@
 F 0 "D2" H 7050 4600 50  0000 C CNN
 F 1 "1N4004" H 7050 4400 50  0000 C CNN
-F 2 "" H 7050 4500 50  0001 C CNN
+F 2 "Diode_THT:D_DO-41_SOD81_P2.54mm_Vertical_AnodeUp" H 7050 4500 50  0001 C CNN
 F 3 "" H 7050 4500 50  0001 C CNN
 F 4 "MC01W08051180R" H 7050 4500 50  0001 C CNN "P/N"
@@
 F 0 "D4" H 7050 5300 50  0000 C CNN
 F 1 "1N4004" H 7050 5100 50  0000 C CNN
-F 2 "" H 7050 5200 50  0001 C CNN
+F 2 "Diode_THT:D_DO-41_SOD81_P2.54mm_Vertical_AnodeUp" H 7050 5200 50  0001 C CNN
 F 3 "" H 7050 5200 50  0001 C CNN
 F 4 "MC01W08051180R" H 7050 5200 50  0001 C CNN "P/N"
@@
 F 0 "C5" H 8125 4350 50  0000 L CNN
 F 1 "100uF/25V" V 7950 4000 50  0000 L CNN
-F 2 "" H 8138 4100 50  0001 C CNN
+F 2 "Capacitor_THT:CP_Radial_D6.3mm_P2.50mm" H 8138 4100 50  0001 C CNN
 F 3 "" H 8100 4250 50  0001 C CNN
 	1    8100 4250
@@
 F 0 "C6" H 9025 4350 50  0000 L CNN
 F 1 "100uF/25V" V 8850 4050 50  0000 L CNN
-F 2 "" H 9038 4100 50  0001 C CNN
+F 2 "Capacitor_THT:CP_Radial_D6.3mm_P2.50mm" H 9038 4100 50  0001 C CNN
 F 3 "" H 9000 4250 50  0001 C CNN
 	1    9000 4250
@@
 F 0 "C1" H 9825 3450 50  0000 L CNN
 F 1 "22uF/16V" V 9650 3150 50  0000 L CNN
-F 2 "" H 9838 3200 50  0001 C CNN
+F 2 "Capacitor_THT:CP_Radial_D5.0mm_P2.50mm" H 9838 3200 50  0001 C CNN
 F 3 "" H 9800 3350 50  0001 C CNN
 	1    9800 3350
@@
 F 0 "C2" H 10175 3450 50  0000 L CNN
 F 1 "100nF" V 10300 3200 50  0000 L CNN
-F 2 "" H 10188 3200 50  0001 C CNN
+F 2 "Capacitor_THT:C_Disc_D4.3mm_W1.9mm_P5.00mm" H 10188 3200 50  0001 C CNN
 F 3 "" H 10150 3350 50  0001 C CNN
 	1    10150 3350
@@
 Wire Wire Line
 	9800 2800 9800 3150
-Wire Wire Line
-	9400 3150 9800 3150
 Wire Wire Line
 	10150 3150 10150 3200
@@
 Wire Wire Line
 	2750 6200 3150 6200
+Wire Wire Line
+	9400 3150 9800 3150
 $EndSCHEMATC

Commit message: Desenhando fonte
Parts:
- C3: footprint (none) -> Capacitor_THT:C_Disc_D4.3mm_W1.9mm_P5.00mm
- U2: footprint Package_SO:HTSOP-8-1EP_3.9x4.9mm_P1.27mm_EP2.4x3.2mm -> Package_SO:SOIC-8_3.9x4.9mm_P1.27mm
Changed lines of the file:
@@
 F 0 "U2" H 4150 3600 50  0000 L CNN
 F 1 "NE555" H 4150 2900 50  0000 L CNN
-F 2 "Package_SO:HTSOP-8-1EP_3.9x4.9mm_P1.27mm_EP2.4x3.2mm" H 4550 3250 50  0001 C CNN
+F 2 "Package_SO:SOIC-8_3.9x4.9mm_P1.27mm" H 4550 3250 50  0001 C CNN
 F 3 "" H 4550 3250 50  0001 C CNN
 	1    4550 3250
@@
 F 0 "C3" H 3625 4000 50  0000 L CNN
 F 1 "10nF" H 3625 3800 50  0000 L CNN
-F 2 "" H 3638 3750 50  0001 C CNN
+F 2 "Capacitor_THT:C_Disc_D4.3mm_W1.9mm_P5.00mm" H 3638 3750 50  0001 C CNN
 F 3 "Falta" H 3600 3900 50  0001 C CNN
 	1    3600 3900
