File: Detector de Metais/detector_metais.kicad_pcb (KiCad board)
At the start: 2 copper layers, 77 parts, among them J1 BARREL_JACK, Q3 BC807-40 ou BC327, Q4 BD911, Q5 BD140, U1 7805, U2 NE555, U3 7905, U4 LM741, U5 4011, U6 NE555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

Commit message: Desenhando fonte
Parts:
- added C3: 10nF, Capacitor_THT:C_Disc_D4.3mm_W1.9mm_P5.00mm, F.Cu at (124.5, 58.4)
- added Q1: BC807-40 ou BC327, Package_TO_SOT_THT:TO-92, F.Cu at (32.3, -30.5)
- added Q2: BF245A, Package_TO_SOT_THT:TO-92, F.Cu at (40.4, -36.5)
- U2: footprint Package_SO:HTSOP-8-1EP_3.9x4.9mm_P1.27mm_EP2.4x3.2mm -> Package_SO:SOIC-8_3.9x4.9mm_P1.27mm
- moved C2 81.7 mm to (104.5, 98.2), turned to 180 degrees
- moved C5 69.8 mm to (120.7, 80.6), turned to 270 degrees
- moved U2 67.5 mm to (118.2, 57.8), turned to 180 degrees
- moved R13 66.1 mm to (168.5, -98.8)
- moved C11 66.1 mm to (159.2, -103.7)
- moved C12 66.1 mm to (159.2, -97.1)
- moved R14 66.1 mm to (163.5, -89.2)
- moved C13 66.1 mm to (169.7, -103.7)
- moved R11 66.1 mm to (158.0, -92.3)
- moved R12 66.1 mm to (158.8, -89.2)
- moved U5 64.6 mm to (175.5, -64.8), turned to 270 degrees
- moved Q3 61.0 mm to (41.3, -2.94)
- moved Q4 60.5 mm to (31.2, -19.3)
- moved D1 56.6 mm to (123.8, 73.7), turned to 270 degrees
- moved C4 56.4 mm to (112.4, 55.9), turned to 270 degrees
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Routing:
- net /555+357/12V: track 0.00 -> 99.7 mm
- net Net-(C7-Pad2): track 0.00 -> 28.9 mm
- net /555+357/+5V: track 0.00 -> 17.7 mm, vias 0 -> 1
- net Net-(C3-Pad1): track 0.00 -> 14.8 mm
- net Net-(C6-Pad1): track 0.00 -> 11.7 mm
- net Net-(C5-Pad1): track 0.00 -> 10.3 mm
- net /555+357/-5V: track 0.00 -> 6.10 mm
- net Net-(C4-Pad1): track 0.00 -> 3.31 mm
- net GND: track 0.00 -> 2.17 mm, vias 0 -> 1
- net Net-(R1-Pad2): track 0.00 -> 1.76 mm
- added copper zone on B.Cu, net Net-(C7-Pad1)
- added copper zone on B.Cu, net Net-(C8-Pad1)
